File: hardware/capibara/capibara.kicad_sch (KiCad schematic)
At the start: 16 parts

Commit message: feat: add final electronic schematic
Connections:
- net 3.3V is gone; now on net +3V3: START1.1, U_BLACKPILL1.20 (3V3)
- net 3,3V renamed +3V3
- net 5V renamed +5V
- net 7.4V renamed +BATT
Other:
- moved on the sheet: BAT1, C1, C2, PWR1, QTR_L1, SHARP1
